File: lab3/PCB Design Lab/PCB Design Lab.kicad_sch (KiCad schematic)
At the start: 0 parts

Commit message: update SCH
Parts:
- added C1: 15pF, Capacitor_SMD:C_0402_1005Metric_Pad0.74x0.62mm_HandSolder, symbol Device:C
- added C2: 2.2µF, Capacitor_SMD:C_0402_1005Metric_Pad0.74x0.62mm_HandSolder, symbol Device:C
- added C3: 1µF, Capacitor_SMD:C_0402_1005Metric_Pad0.74x0.62mm_HandSolder, symbol Device:C
- added C4: 0.01µF, Capacitor_SMD:C_0402_1005Metric_Pad0.74x0.62mm_HandSolder, symbol Device:C
- added C5, C6: 100nF, Capacitor_SMD:C_0402_1005Metric_Pad0.74x0.62mm_HandSolder, symbol Device:C
- added D1: LED, LED_SMD:LED_0402_1005Metric_Pad0.77x0.64mm_HandSolder, symbol Device:LED
- added J1: Conn_01x04_Pin, Connector_PinSocket_2.54mm:PinSocket_1x04_P2.54mm_Vertical, symbol Connector:Conn_01x04_Pin
- added R1: 51k, Resistor_SMD:R_0402_1005Metric_Pad0.72x0.64mm_HandSolder, symbol Device:R
- added R2: 30.1k, Resistor_SMD:R_0402_1005Metric_Pad0.72x0.64mm_HandSolder, symbol Device:R
- added R3, R4: 10k, Resistor_SMD:R_0402_1005Metric_Pad0.72x0.64mm_HandSolder, symbol Device:R
- added R5: 1k, Resistor_SMD:R_0402_1005Metric_Pad0.72x0.64mm_HandSolder, symbol Device:R
- added U1: TPS79301DBVR, TPS79301DBVR:SOT95P280X145-6N, symbol TPS79301DBVR:TPS79301DBVR
- added U2: LSM6DSOXTR, LSM6DSOXTR:PQFN50P250X300X86-14N, symbol LSM6DSOXTR:LSM6DSOXTR
Connections:
- new net: C1.2, R1.2, R2.1, U1.5 (FB)
- new net: D1.2 (A), R5.2
- new net: C4.1, U1.4 (NR)
- new net +3V3: C1.1, C2.1, C5.2, C6.2, R1.1, R3.1, R4.1, R5.1, U1.6 (OUT), U2.12 (CS), U2.5 (VDDIO), U2.8 (VDD)
- new net GND: C2.2, C3.2, C4.2, C5.1, C6.1, D1.1 (K), J1.4 (Pin_4), R2.2, U1.2 (GND), U2.1 (SDO/SA0), U2.2 (SDX), U2.3 (SCX), U2.6 (GND), U2.7 (GND)
- new net SCL: J1.3 (Pin_3), R3.2, U2.13 (SCL)
- new net SDA: J1.2 (Pin_2), R4.2, U2.14 (SDA)
- new net VCC: C3.1, J1.1 (Pin_1), U1.1 (IN), U1.3 (EN)
- no-connect marks 0 -> 4
Other:
- title: (none) -> Lab4-PCB Design Lab
